Commit message: Incorporate the ZED urdf into the kobuki urdf.

File: kobuki_zed_vlp16_ws/workspaces/kobuki_ws/src/kobuki_ros/kobuki_description/urdf/zed/zed_descr.urdf.xacro (robot description, xacro)
@@ -18,8 +18,8 @@
   <xacro:arg name="camera_name"   default="zed" />
   <xacro:arg name="camera_model"  default="zed" />
-  <xacro:include filename="$(find zed_wrapper)/urdf/zed_macro.urdf.xacro" />
+  <xacro:include filename="$(find kobuki_description)/urdf/zed/zed_macro.urdf.xacro" />
   <xacro:zed_camera name="$(arg camera_name)" model="$(arg camera_model)">
   </xacro:zed_camera>
-  <xacro:include filename="$(find zed_wrapper)/urdf/zed_gazebo.urdf.xacro" />
+  <xacro:include filename="$(find kobuki_description)/urdf/zed/zed_gazebo.urdf.xacro" />
   <xacro:zed_gazebo name="$(arg camera_name)" />
 </robot>

File: kobuki_zed_vlp16_ws/workspaces/kobuki_ws/src/kobuki_ros/kobuki_description/urdf/zed/zed_macro.urdf.xacro (robot description, xacro)
@@ -16,5 +16,5 @@
 -->
 <robot xmlns:xacro="http://wiki.ros.org/xacro">
-  <xacro:include filename="$(find zed_wrapper)/urdf/include/materials.urdf.xacro" />
+  <xacro:include filename="$(find kobuki_description)/urdf/zed/include/materials.urdf.xacro" />
   <xacro:property name="M_PI"     value="3.1415926535897931" />
   <!--
@@ -85,5 +85,5 @@
         <origin xyz="${screw_offset_x} 0 ${screw_offset_z}" rpy="0 0 0"/>
         <geometry>
-          <mesh filename="package://zed_interfaces/meshes/${model}.stl" />
+          <mesh filename="package://kobuki_description/meshes/zed/${model}.stl" />
         </geometry>
         <material name="${model}_mat" />
@@ -91,5 +91,5 @@
       <collision>
         <geometry>
-          <mesh filename="package://zed_interfaces/meshes/${model}.stl" />
+          <mesh filename="package://kobuki_description/meshes/zed/${model}.stl" />
         </geometry>
       </collision>
